Commit message: working robots + manipulators

File: arena_robots/arena_robots/robots/boxer/urdf/boxer.urdf.xacro (robot description, xacro)
@@ -119,7 +119,8 @@
   <xacro:include filename="$(find arena_robots)/robots/boxer/urdf/include/sensors.urdf.xacro" />
   <xacro:include filename="$(find arena_robots)/robots/boxer/urdf/include/wheels_and_casters.urdf.xacro" />
+  <xacro:include filename="$(find arena_robots)/robots/boxer/urdf/base_hw/boxer.ros2_control.urdf" />
+  <xacro:include filename="$(find arena_robots)/robots/boxer/urdf/boxer.gazebo" />
+  <xacro:boxer_base_hw_controller/>
   <!-- User extensions -->
   <xacro:include filename="$(optenv BOXER_URDF_EXTRAS empty.urdf)" />
-  <!-- Bring in simulation data for Gazebo. -->
-  <xacro:include filename="$(find arena_robots)/robots/boxer/urdf/boxer.gazebo" />
 </robot>

File: arena_robots/arena_robots/robots/boxer/urdf/include/sensors.urdf.xacro (robot description, xacro)
@@ -29,5 +29,5 @@
     <turnGravityOff>true</turnGravityOff>
     <sensor type="depth" name="realsense_front_camera">
-      <gz_frame_id>$(arg name)/realsense_front_camera_link</gz_frame_id>
+      <gz_frame_id>$(arg sim_path)/realsense_front_camera_link</gz_frame_id>
       <update_rate>30</update_rate>
       <camera>
@@ -91,5 +91,5 @@
     <turnGravityOff>true</turnGravityOff>
     <sensor type="gpu_lidar" name="front_laser">
-      <gz_frame_id>$(arg name)/front_laser</gz_frame_id>
+      <gz_frame_id>$(arg sim_path)/front_laser</gz_frame_id>
       <pose>0 0 0 0 0 0</pose>
       <visualize>false</visualize>
@@ -142,5 +142,5 @@
     <turnGravityOff>true</turnGravityOff>
     <sensor type="gpu_lidar" name="rear_laser">
-      <gz_frame_id>$(arg name)/rear_sensor</gz_frame_id>
+      <gz_frame_id>$(arg sim_path)/rear_sensor</gz_frame_id>
       <pose>0 0 0 0 0 0</pose>
       <visualize>false</visualize>

File: arena_robots/arena_robots/robots/dingo/urdf/dingo-d.urdf.xacro (robot description, xacro)
@@ -221,4 +221,6 @@
   <xacro:include filename="$(find arena_robots)/robots/dingo/urdf/pacs.urdf.xacro"/>
   <xacro:pacs/>
+  <!-- ros2_control hardware block (diff drive, DINGO_OMNI=0 only). -->
+  <xacro:include filename="$(find arena_robots)/robots/dingo/urdf/base_hw/dingo.ros2_control.urdf" />
   <!-- Bring in simulation data for Gazebo. -->
   <xacro:include filename="$(find arena_robots)/robots/dingo/urdf/dingo.gazebo" />
@@ -229,3 +231,4 @@
   <!-- Optional custom includes. -->
   <xacro:include filename="$(optenv DINGO_URDF_EXTRAS empty.urdf)" />
+  <xacro:dingo_base_hw_controller/>
 </robot>

File: arena_robots/arena_robots/robots/husky/urdf/husky.urdf.xacro (robot description, xacro)
@@ -125,4 +125,6 @@
   <xacro:include filename="$(find arena_robots)/robots/husky/urdf/decorations.urdf.xacro" />
   <xacro:include filename="$(find arena_robots)/robots/husky/urdf/wheel.urdf.xacro" />
+  <xacro:include filename="$(find arena_robots)/robots/husky/urdf/base_hw/husky.ros2_control.urdf" />
+  <xacro:include filename="$(find arena_robots)/robots/husky/urdf/husky.gazebo" />
   <xacro:property name="M_PI" value="3.14159"/>
   <!-- Base Size -->
@@ -323,10 +325,5 @@
     <xacro:outdoornav_sensors outdoornav_configuration="$(arg outdoornav_configuration)" />
   </xacro:if>
-  <gazebo>
-    <plugin name="gazebo_ros_control" filename="libgazebo_ros_control.so">
-      <robotNamespace>$(arg robot_namespace)</robotNamespace>
-      <legacyModeNS>true</legacyModeNS>
-    </plugin>
-  </gazebo>
+  <xacro:husky_base_hw_controller/>
   <gazebo>
     <plugin name="imu_controller" filename="libhector_gazebo_ros_imu.so">

File: arena_robots/arena_robots/robots/husky/urdf/wheel.urdf.xacro (robot description, xacro)
@@ -43,11 +43,11 @@
 		</link>
 		<gazebo reference="${wheel_prefix}_wheel_link">
-			<mu1 value="1.0"/>
-			<mu2 value="1.0"/>
-			<kp value="10000000.0" />
-			<kd value="1.0" />
-			<fdir1 value="1 0 0"/>
+			<mu1>1.0</mu1>
+			<mu2>0.5</mu2>
+			<kp>10000000.0</kp>
+			<kd>1.0</kd>
+			<fdir1>1 0 0</fdir1>
 		</gazebo>
-		<joint name="${wheel_prefix}_wheel" type="continuous">
+		<joint name="${wheel_prefix}_wheel_joint" type="continuous">
 			<parent link="base_link"/>
 			<child link="${wheel_prefix}_wheel_link"/>
@@ -60,5 +60,5 @@
 				<mechanicalReduction>1</mechanicalReduction>
 			</actuator>
-			<joint name="${wheel_prefix}_wheel">
+			<joint name="${wheel_prefix}_wheel_joint">
 				<hardwareInterface>hardware_interface/VelocityJointInterface</hardwareInterface>
 			</joint>

File: arena_robots/arena_robots/robots/jackal/urdf/jackal.urdf.xacro (robot description, xacro)
@@ -1,8 +1,8 @@
 <?xml version="1.0"?>
 <robot name="jackal" xmlns:xacro="http://www.ros.org/wiki/xacro">
-  <xacro:arg name="is_sim" default="false" />
   <xacro:arg name="prefix" default="" />
   <xacro:arg name="sim_path" default="" />
-  <xacro:arg name="gazebo_controllers" default="$(find jackal_control)/config/control.yaml" />
+  <xacro:arg name="namespace" default="" />
+  <xacro:arg name="gazebo_controllers" default="" />
   <xacro:property name="PI" value="3.1415926535897931" />
   <xacro:property name="wheelbase" value="0.262" />
@@ -254,36 +254,6 @@
     <origin xyz="${mount_spacing} 0 0" />
   </joint>
-  <!-- ROS2 controls -->
-  <ros2_control name="jackal_hardware" type="system">
-    <hardware>
-      <xacro:if value="$(arg is_sim)">
-        <plugin>gazebo_ros2_control/GazeboSystem</plugin>
-      </xacro:if>
-      <xacro:unless value="$(arg is_sim)">
-        <plugin>jackal_hardware/JackalHardware</plugin>
-        <plugin>fake_components/GenericSystem</plugin>
-      </xacro:unless>
-    </hardware>
-    <joint name="front_left_wheel_joint">
-      <command_interface name="velocity"/>
-      <state_interface name="position"/>
-      <state_interface name="velocity"/>
-    </joint>
-    <joint name="rear_left_wheel_joint">
-      <command_interface name="velocity"/>
-      <state_interface name="position"/>
-      <state_interface name="velocity"/>
-    </joint>
-    <joint name="front_right_wheel_joint">
-      <command_interface name="velocity"/>
-      <state_interface name="position"/>
-      <state_interface name="velocity"/>
-    </joint>
-    <joint name="rear_right_wheel_joint">
-      <command_interface name="velocity"/>
-      <state_interface name="position"/>
-      <state_interface name="velocity"/>
-    </joint>
-  </ros2_control>
+  <xacro:include filename="$(find arena_robots)/robots/jackal/urdf/base_hw/jackal.ros2_control.urdf" />
+  <xacro:jackal_base_hw_controller/>
   <!-- Bring in simulation data for Gazebo. -->
   <xacro:include filename="./jackal.gazebo" />

File: arena_robots/arena_robots/robots/rbkairos/urdf/rbkairos.urdf.xacro (robot description, xacro)
@@ -7,6 +7,5 @@
   <xacro:include filename="$(find arena_robots)/robots/rbkairos/urdf/bases/rbkairos/rbkairos_base.urdf.xacro" />
   <xacro:include filename="$(find arena_robots)/robots/rbkairos/urdf/base_hw/rbkairos.ros2_control.urdf" />
-  <xacro:include filename="$(find arena_robots)/robots/rbkairos/simulators/gazebo_classic/rbkairos/rbkairos_control.urdf.xacro" />
-  <xacro:include filename="$(find arena_robots)/robots/rbkairos/simulators/gazebo_ignition/rbkairos/rbkairos_control.urdf.xacro" />
+  <xacro:include filename="$(find arena_robots)/robots/rbkairos/urdf/rbkairos.gazebo" />
   <xacro:include filename="$(find arena_robots)/robots/rbkairos/urdf/all_sensors.urdf.xacro" />
   <!-- Properties and Arguments -->
@@ -14,5 +13,6 @@
   <xacro:arg name="prefix" default="robot_"/>
   <xacro:arg name="gazebo_classic" default="false"/>
-  <xacro:arg name="gazebo_ignition" default="false"/>
+  <xacro:arg name="gazebo_ignition" default="true"/>
+  <xacro:arg name="gazebo_controllers" default=""/>
   <xacro:property name="front_laser_offset_x" value="0.42109"/>
   <xacro:property name="front_laser_offset_y" value="-0.32737"/>
@@ -71,24 +71,6 @@
     <xacro:ros_planar_move_gazebo_classic/>
   </xacro:if>
-  <xacro:if value="$(arg gazebo_ignition)">
-    <xacro:rbkairos_gz_ignition_control namespace="$(arg namespace)" prefix="$(arg prefix)"/>
-  </xacro:if>
   <xacro:unless value="$(arg gazebo_classic)">
-    <xacro:unless value="$(arg gazebo_ignition)">
-      <xacro:rbkairos_base_hw_controller/>
-    </xacro:unless>
+    <xacro:rbkairos_base_hw_controller/>
   </xacro:unless>
-  <gazebo>
-    <plugin
-      filename="gz-sim-pose-publisher-system"
-      name="gz::sim::systems::PosePublisher">
-      <publish_model_pose>true</publish_model_pose>
-      <publish_link_pose>false</publish_link_pose>
-      <publish_collision_pose>false</publish_collision_pose>
-      <publish_visual_pose>false</publish_visual_pose>
-      <publish_sensor_pose>false</publish_sensor_pose>
-      <publish_nested_model_pose>true</publish_nested_model_pose>
-      <use_pose_vector_msg>false</use_pose_vector_msg>
-    </plugin>
-  </gazebo>
 </robot>

File: arena_robots/arena_robots/robots/rbkairos_plus/urdf/rbkairos_plus.urdf.xacro (robot description, xacro)
@@ -7,6 +7,5 @@
   <xacro:include filename="$(find arena_robots)/robots/rbkairos/urdf/bases/rbkairos/rbkairos_base.urdf.xacro" />
   <xacro:include filename="$(find arena_robots)/robots/rbkairos_plus/urdf/base_hw/rbkairos_plus.ros2_control.urdf" />
-  <xacro:include filename="$(find arena_robots)/robots/rbkairos/simulators/gazebo_classic/rbkairos/rbkairos_control.urdf.xacro" />
-  <xacro:include filename="$(find arena_robots)/robots/rbkairos/simulators/gazebo_ignition/rbkairos/rbkairos_control.urdf.xacro" />
+  <xacro:include filename="$(find arena_robots)/robots/rbkairos_plus/urdf/rbkairos_plus.gazebo" />
   <xacro:include filename="$(find arena_robots)/robots/rbkairos/urdf/all_sensors.urdf.xacro" />
   <xacro:include filename="$(find ur_description)/urdf/ur_macro.xacro" />
@@ -15,5 +14,6 @@
   <xacro:arg name="prefix" default="robot_"/>
   <xacro:arg name="gazebo_classic" default="false"/>
-  <xacro:arg name="gazebo_ignition" default="false"/>
+  <xacro:arg name="gazebo_ignition" default="true"/>
+  <xacro:arg name="gazebo_controllers" default=""/>
   <xacro:arg name="ur_type" default="ur5e"/>
   <xacro:arg name="joint_limit_params" default="$(find ur_description)/config/$(arg ur_type)/joint_limits.yaml"/>
@@ -92,11 +92,6 @@
     <xacro:ros_planar_move_gazebo_classic/>
   </xacro:if>
-  <xacro:if value="$(arg gazebo_ignition)">
-    <xacro:rbkairos_gz_ignition_control namespace="$(arg namespace)" prefix="$(arg prefix)"/>
-  </xacro:if>
   <xacro:unless value="$(arg gazebo_classic)">
-    <xacro:unless value="$(arg gazebo_ignition)">
-      <xacro:rbkairos_base_hw_controller/>
-    </xacro:unless>
+    <xacro:rbkairos_plus_arm_hw_controller/>
   </xacro:unless>
 </robot>

File: arena_robots/arena_robots/robots/rbrobout/urdf/rbrobout.urdf.xacro (robot description, xacro)
@@ -4,15 +4,13 @@
   <!-- Imported elements -->
   <!-- ***************** -->
-  <!-- Import all posible elements defined in the urdf.xacro files. All these elements are defined as macro:xacros -->
   <xacro:include filename="$(find arena_robots)/robots/rbrobout/urdf/bases/rbrobout/rbrobout_base.urdf.xacro" />
   <xacro:include filename="$(find arena_robots)/robots/rbrobout/urdf/base_hw/rbrobout.ros2_control.urdf" />
-  <xacro:include filename="$(find arena_robots)/robots/rbrobout/simulators/gazebo_classic/rbrobout/rbrobout_control.urdf.xacro" />
-  <xacro:include filename="$(find arena_robots)/robots/rbrobout/simulators/gazebo_ignition/rbrobout/rbrobout_control.urdf.xacro" />
+  <xacro:include filename="$(find arena_robots)/robots/rbrobout/urdf/rbrobout.gazebo" />
   <xacro:include filename="$(find arena_robots)/robots/rbrobout/urdf/all_sensors.urdf.xacro" />
   <!-- Properties and Arguments -->
   <xacro:arg name="namespace" default="robot"/>
   <xacro:arg name="prefix" default="robot_"/>
-  <xacro:arg name="gazebo_classic" default="false"/>
-  <xacro:arg name="gazebo_ignition" default="false"/>
+  <xacro:arg name="gazebo_ignition" default="true"/>
+  <xacro:arg name="gazebo_controllers" default=""/>
   <xacro:property name="front_laser_offset_x" value="0.8"/>
   <xacro:property name="front_laser_offset_y" value="0.366"/>
@@ -24,59 +22,35 @@
   <xacro:property name="imu_offset_y" value="-0.3"/>
   <xacro:property name="imu_offset_z" value="0.0725"/>
-  <xacro:rbrobout prefix="$(arg prefix)" gazebo_classic="$(arg gazebo_classic)" gazebo_ignition="$(arg gazebo_ignition)"/>
+  <xacro:rbrobout prefix="$(arg prefix)" gazebo_ignition="$(arg gazebo_ignition)"/>
   <!-- IMU -->
-    <xacro:sensor_vectornav
-        frame_prefix="$(arg prefix)vectornav_"
-        parent="$(arg prefix)base_link"
-        node_namespace="$(arg namespace)"
-        gazebo_classic="$(arg gazebo_classic)"
-        gazebo_ignition="$(arg gazebo_ignition)">
-        <origin xyz="${imu_offset_x} ${imu_offset_y} ${imu_offset_z}" rpy="0 0 0"/>
-    </xacro:sensor_vectornav>
+  <xacro:sensor_vectornav
+      frame_prefix="$(arg prefix)vectornav_"
+      parent="$(arg prefix)base_link"
+      node_namespace="$(arg namespace)"
+      gazebo_classic="false"
+      gazebo_ignition="$(arg gazebo_ignition)">
+      <origin xyz="${imu_offset_x} ${imu_offset_y} ${imu_offset_z}" rpy="0 0 0"/>
+  </xacro:sensor_vectornav>
   <!-- 2d laser -->
-    <xacro:sensor_sick_microscan3
-        frame_prefix="$(arg prefix)front_laser_"
-        parent="$(arg prefix)base_link"
-        node_namespace="$(arg namespace)"
-        node_name="front_laser"
-        gazebo_classic="$(arg gazebo_classic)"
-        gazebo_ignition="$(arg gazebo_ignition)">
-        <origin xyz="${front_laser_offset_x} ${front_laser_offset_y} ${front_laser_offset_z}" rpy="0 0 ${1/4*PI}"/>
-    </xacro:sensor_sick_microscan3>
-    <!-- 2d laser -->
-    <xacro:sensor_sick_microscan3
-        frame_prefix="$(arg prefix)rear_laser_"
-        parent="$(arg prefix)base_link"
-        node_namespace="$(arg namespace)"
-        node_name="rear_laser"
-        gazebo_classic="$(arg gazebo_classic)"
-        gazebo_ignition="$(arg gazebo_ignition)">
-        <origin xyz="${rear_laser_offset_x} ${rear_laser_offset_y} ${rear_laser_offset_z}" rpy="0 0 ${-3/4*PI}"/>
-    </xacro:sensor_sick_microscan3>
-    <!-- Controllers -->
-    <xacro:if value="$(arg gazebo_classic)">
-        <xacro:rbrobout_gz_classic_control namespace="$(arg namespace)" prefix="$(arg prefix)"/>
-        <xacro:ros_planar_move_gazebo_classic/>
-    </xacro:if>
-    <xacro:if value="$(arg gazebo_ignition)">
-        <xacro:rbrobout_gz_ignition_control namespace="$(arg namespace)" prefix="$(arg prefix)"/>
-    </xacro:if>
-    <xacro:unless value="$(arg gazebo_classic)">
-        <xacro:unless value="$(arg gazebo_ignition)">
-            <xacro:rbrobout_base_hw_controller/>
-        </xacro:unless>
-    </xacro:unless>
-    <gazebo>
-        <plugin
-        filename="gz-sim-pose-publisher-system"
-        name="gz::sim::systems::PosePublisher">
-        <publish_model_pose>true</publish_model_pose>
-        <publish_link_pose>false</publish_link_pose>
-        <publish_collision_pose>false</publish_collision_pose>
-        <publish_visual_pose>false</publish_visual_pose>
-        <publish_sensor_pose>false</publish_sensor_pose>
-        <publish_nested_model_pose>true</publish_nested_model_pose>
-        <use_pose_vector_msg>false</use_pose_vector_msg>
-        </plugin>
-    </gazebo>
+  <xacro:sensor_sick_microscan3
+      frame_prefix="$(arg prefix)front_laser_"
+      parent="$(arg prefix)base_link"
+      node_namespace="$(arg namespace)"
+      node_name="front_laser"
+      gazebo_classic="false"
+      gazebo_ignition="$(arg gazebo_ignition)">
+      <origin xyz="${front_laser_offset_x} ${front_laser_offset_y} ${front_laser_offset_z}" rpy="0 0 ${1/4*PI}"/>
+  </xacro:sensor_sick_microscan3>
+  <!-- 2d laser -->
+  <xacro:sensor_sick_microscan3
+      frame_prefix="$(arg prefix)rear_laser_"
+      parent="$(arg prefix)base_link"
+      node_namespace="$(arg namespace)"
+      node_name="rear_laser"
+      gazebo_classic="false"
+      gazebo_ignition="$(arg gazebo_ignition)">
+      <origin xyz="${rear_laser_offset_x} ${rear_laser_offset_y} ${rear_laser_offset_z}" rpy="0 0 ${-3/4*PI}"/>
+  </xacro:sensor_sick_microscan3>
+  <!-- ros2_control hardware block (always active; gz plugin loaded via rbrobout.gazebo) -->
+  <xacro:rbrobout_base_hw_controller/>
 </robot>

File: arena_robots/arena_robots/robots/rbrobout_plus/urdf/rbrobout_plus.urdf.xacro (robot description, xacro)
@@ -7,7 +7,8 @@
   <xacro:include filename="$(find arena_robots)/robots/rbrobout/urdf/bases/rbrobout/rbrobout_base.urdf.xacro" />
   <xacro:include filename="$(find arena_robots)/robots/rbrobout/urdf/bases/rbrobout/rbrobout_top_cover.urdf.xacro" />
+  <!-- Arena ros2_control block (arm + lift). Top-level, no macro. -->
   <xacro:include filename="$(find arena_robots)/robots/rbrobout_plus/urdf/base_hw/rbrobout_plus.ros2_control.urdf" />
-  <xacro:include filename="$(find arena_robots)/robots/rbrobout/simulators/gazebo_classic/rbrobout/rbrobout_control.urdf.xacro" />
-  <xacro:include filename="$(find arena_robots)/robots/rbrobout/simulators/gazebo_ignition/rbrobout/rbrobout_control.urdf.xacro" />
+  <!-- gz_ros2_control plugin (loads control.yaml, namespace + path via xacro args) -->
+  <xacro:include filename="$(find arena_robots)/robots/rbrobout_plus/urdf/rbrobout_plus.gazebo" />
   <xacro:include filename="$(find arena_robots)/robots/rbrobout/urdf/all_sensors.urdf.xacro" />
   <xacro:include filename="$(find ur_description)/urdf/ur_macro.xacro" />
@@ -17,5 +18,9 @@
   <xacro:arg name="prefix" default="robot_"/>
   <xacro:arg name="gazebo_classic" default="false"/>
-  <xacro:arg name="gazebo_ignition" default="false"/>
+  <xacro:arg name="gazebo_ignition" default="true"/>
+  <!-- When true, fall back to legacy rbrobout_gz_ignition_control (its own ros2_control + plugin).
+       Default false so Arena's ros2_control bringup (arm + lift via MoveIt) is active. -->
+  <xacro:arg name="use_legacy_controllers" default="false"/>
+  <xacro:arg name="gazebo_controllers" default=""/>
   <xacro:arg name="ur_type" default="ur10e"/>
   <xacro:arg name="joint_limit_params" default="$(find ur_description)/config/$(arg ur_type)/joint_limits.yaml"/>
@@ -92,5 +97,7 @@
     </xacro:if>
     <xacro:if value="$(arg gazebo_ignition)">
-        <xacro:rbrobout_gz_ignition_control namespace="$(arg namespace)" prefix="$(arg prefix)"/>
+        <xacro:if value="$(arg use_legacy_controllers)">
+            <xacro:rbrobout_gz_ignition_control namespace="$(arg namespace)" prefix="$(arg prefix)"/>
+        </xacro:if>
     </xacro:if>
     <xacro:unless value="$(arg gazebo_classic)">

File: arena_robots/arena_robots/robots/rbsummit/urdf/rbsummit.urdf.xacro (robot description, xacro)
@@ -7,7 +7,6 @@
 	<!-- Import summit XL macro -->
 	<xacro:include filename="$(find arena_robots)/robots/rbsummit/urdf/bases/rbsummit/rbsummit_base.xacro"/>
-    <xacro:include filename="$(find arena_robots)/robots/rbsummit/urdf/base_hw/rbsummit.ros2_control.urdf" />
-	<xacro:include filename="$(find arena_robots)/robots/rbsummit/simulators/gazebo_classic/rbsummit/rbsummit_control.urdf.xacro"/>
-	<xacro:include filename="$(find arena_robots)/robots/rbsummit/simulators/gazebo_ignition/rbsummit/rbsummit_control.urdf.xacro"/>
+	<xacro:include filename="$(find arena_robots)/robots/rbsummit/urdf/base_hw/rbsummit.ros2_control.urdf" />
+	<xacro:include filename="$(find arena_robots)/robots/rbsummit/urdf/rbsummit.gazebo" />
 	<!-- Import all available sensors -->
 	<xacro:include filename="$(find arena_robots)/robots/rbsummit/urdf/all_sensors.urdf.xacro" />
@@ -86,13 +85,8 @@
     <xacro:if value="$(arg gazebo_classic)">
       <xacro:rbsummit_gz_classic_control namespace="$(arg namespace)" prefix="$(arg prefix)"/>
-        <xacro:ros_planar_move_gazebo_classic/>
-    </xacro:if>
-    <xacro:if value="$(arg gazebo_ignition)">
-      <xacro:rbsummit_gz_ignition_control namespace="$(arg namespace)" prefix="$(arg prefix)"/>
+      <xacro:ros_planar_move_gazebo_classic/>
     </xacro:if>
     <xacro:unless value="$(arg gazebo_classic)">
-      <xacro:unless value="$(arg gazebo_ignition)">
-        <xacro:rbsummit_base_hw_controller/>
-      </xacro:unless>
+      <xacro:rbsummit_base_hw_controller/>
     </xacro:unless>
 	<gazebo>

File: arena_robots/arena_robots/robots/rbtheron/urdf/rbtheron.urdf.xacro (robot description, xacro)
@@ -8,7 +8,6 @@
 	<!-- Import rbtheron macro -->
 	<xacro:include filename="$(find arena_robots)/robots/rbtheron/urdf/bases/rbtheron/rbtheron_base.xacro"/>
-    <xacro:include filename="$(find arena_robots)/robots/rbtheron/urdf/base_hw/rbtheron.ros2_control.urdf" />
-	<xacro:include filename="$(find arena_robots)/robots/rbtheron/simulators/gazebo_classic/rbtheron/rbtheron_control.urdf.xacro"/>
-	<xacro:include filename="$(find arena_robots)/robots/rbtheron/simulators/gazebo_ignition/rbtheron/rbtheron_control.urdf.xacro"/>
+	<xacro:include filename="$(find arena_robots)/robots/rbtheron/urdf/base_hw/rbtheron.ros2_control.urdf" />
+	<xacro:include filename="$(find arena_robots)/robots/rbtheron/urdf/rbtheron.gazebo" />
 	<!-- Import all available sensors -->
 	<xacro:include filename="$(find arena_robots)/robots/rbtheron/urdf/all_sensors.urdf.xacro" />
@@ -24,4 +23,5 @@
 	<xacro:arg name="gazebo_classic" default="false"/>
 	<xacro:arg name="gazebo_ignition" default="false"/>
+	<xacro:arg name="gazebo_controllers" default=""/>
 	<!-- Here we create the robot using the xacro:macro imported at the beggining of this file -->
 	<xacro:rbtheron prefix="$(arg prefix)" hq="${hq}"/>
@@ -94,12 +94,5 @@
         <xacro:ros_planar_move_gazebo_classic/>
 	</xacro:if>
-	<xacro:if value="$(arg gazebo_ignition)">
-		<xacro:rbtheron_gz_ignition_control namespace="$(arg namespace)" prefix="$(arg prefix)"/>
-	</xacro:if>
-    <xacro:unless value="$(arg gazebo_classic)">
-        <xacro:unless value="$(arg gazebo_ignition)">
-            <xacro:rbtheron_base_hw_controller/>
-        </xacro:unless>
-    </xacro:unless>
+	<xacro:rbtheron_base_hw_controller/>
     <gazebo>
         <plugin
