Commit message: working robots + manipulators

File: arena_robots/arena_robots/robots/rbvogui/urdf/rbvogui.urdf.xacro (robot description, xacro)
@@ -9,6 +9,5 @@
     <xacro:include filename="$(find arena_robots)/robots/rbvogui/urdf/bases/rbvogui/rbvogui_base.urdf.xacro" />
     <xacro:include filename="$(find arena_robots)/robots/rbvogui/urdf/base_hw/rbvogui.ros2_control.urdf" />
-    <xacro:include filename="$(find arena_robots)/robots/rbvogui/simulators/gazebo_classic/rbvogui/rbvogui_control.urdf.xacro" />
-    <xacro:include filename="$(find arena_robots)/robots/rbvogui/simulators/gazebo_ignition/rbvogui/rbvogui_control.urdf.xacro" />
+    <xacro:include filename="$(find arena_robots)/robots/rbvogui/urdf/rbvogui.gazebo" />
     <!-- Import all available sensors -->
     <xacro:include filename="$(find arena_robots)/robots/rbvogui/urdf/all_sensors.urdf.xacro" />
@@ -18,6 +17,5 @@
 	<xacro:arg name="namespace" default="robot"/>
 	<xacro:arg name="prefix" default="robot_"/>
-	<xacro:arg name="gazebo_classic" default="false"/>
-	<xacro:arg name="gazebo_ignition" default="false"/>
+	<xacro:arg name="gazebo_controllers" default=""/>
     <xacro:rbvogui prefix="$(arg prefix)" hq="${hq}"/>
     <!-- SENSORS see robotnik_sensors for the specific configuration -->
@@ -27,6 +25,6 @@
         parent="$(arg prefix)chassis_link"
         node_namespace="$(arg namespace)"
-        gazebo_classic="$(arg gazebo_classic)"
-        gazebo_ignition="$(arg gazebo_ignition)">
+        gazebo_classic="false"
+        gazebo_ignition="true">
         <origin xyz="0.3 -0.3 0.0725" rpy="0 0 0"/>
     </xacro:sensor_vectornav>
@@ -37,6 +35,6 @@
         node_namespace="$(arg namespace)"
         node_name="front_camera"
-        gazebo_classic="$(arg gazebo_classic)"
-        gazebo_ignition="$(arg gazebo_ignition)">
+        gazebo_classic="false"
+        gazebo_ignition="true">
         <origin xyz="0.46462 0.0 0.18258" rpy="0 0 0"/>
     </xacro:sensor_intel_realsense_d435>
@@ -47,6 +45,6 @@
         node_namespace="$(arg namespace)"
         node_name="rear_camera"
-        gazebo_classic="$(arg gazebo_classic)"
-        gazebo_ignition="$(arg gazebo_ignition)">
+        gazebo_classic="false"
+        gazebo_ignition="true">
         <origin xyz="-0.503 0.0 0.29" rpy="0 0 -${PI}"/>
     </xacro:sensor_intel_realsense_d435>
@@ -57,6 +55,6 @@
         node_namespace="$(arg namespace)"
         node_name="front_laser"
-        gazebo_classic="$(arg gazebo_classic)"
-        gazebo_ignition="$(arg gazebo_ignition)">
+        gazebo_classic="false"
+        gazebo_ignition="true">
         <origin xyz="0.53 0.33 0.1145" rpy="${PI} 0 ${PI/4}"/>
     </xacro:sensor_sick_s300>
@@ -66,33 +64,9 @@
         node_namespace="$(arg namespace)"
         node_name="rear_laser"
-        gazebo_classic="$(arg gazebo_classic)"
-        gazebo_ignition="$(arg gazebo_ignition)">
+        gazebo_classic="false"
+        gazebo_ignition="true">
         <origin xyz="-0.53 -0.33 0.1145" rpy="${PI} 0 ${-PI*3/4}"/>
     </xacro:sensor_sick_s300>
-	<!-- Controllers -->
-	<xacro:if value="$(arg gazebo_classic)">
-		<xacro:rbvogui_gz_classic_control namespace="$(arg namespace)" prefix="$(arg prefix)"/>
-        <xacro:ros_planar_move_gazebo_classic/>
-	</xacro:if>
-	<xacro:if value="$(arg gazebo_ignition)">
-		<xacro:rbvogui_gz_ignition_control namespace="$(arg namespace)" prefix="$(arg prefix)"/>
-	</xacro:if>
-    <xacro:unless value="$(arg gazebo_classic)">
-        <xacro:unless value="$(arg gazebo_ignition)">
-            <xacro:rbvogui_base_hw_controller/>
-        </xacro:unless>
-    </xacro:unless>
-    <gazebo>
-        <plugin
-        filename="gz-sim-pose-publisher-system"
-        name="gz::sim::systems::PosePublisher">
-        <publish_model_pose>true</publish_model_pose>
-        <publish_link_pose>false</publish_link_pose>
-        <publish_collision_pose>false</publish_collision_pose>
-        <publish_visual_pose>false</publish_visual_pose>
-        <publish_sensor_pose>false</publish_sensor_pose>
-        <publish_nested_model_pose>true</publish_nested_model_pose>
-        <use_pose_vector_msg>false</use_pose_vector_msg>
-        </plugin>
-    </gazebo>
+    <!-- ros2_control block (gz_ros2_control/GazeboSimSystem) and PosePublisher loaded via rbvogui.gazebo -->
+    <xacro:rbvogui_base_hw_controller/>
 </robot>

File: arena_robots/arena_robots/robots/rbvogui_plus/urdf/rbvogui_plus.urdf.xacro (robot description, xacro)
@@ -1,4 +1,10 @@
 <?xml version="1.0"?>
 <robot name="rbvogui_plus" xmlns:xacro="http://wiki.ros.org/xacro">
+  <xacro:arg name="namespace" default=""/>
+  <xacro:arg name="prefix" default="robot_"/>
+  <xacro:arg name="gazebo_controllers" default=""/>
   <xacro:include filename="$(find robotnik_description)/robots/rbvogui/rbvogui_plus.urdf.xacro"/>
+  <xacro:include filename="$(find arena_robots)/robots/rbvogui_plus/urdf/base_hw/rbvogui_plus.ros2_control.urdf"/>
+  <!-- gz_ros2_control plugin (loads control.yaml; namespace + path set via xacro args) -->
+  <xacro:include filename="$(find arena_robots)/robots/rbvogui_plus/urdf/rbvogui_plus.gazebo"/>
 </robot>

File: arena_robots/arena_robots/robots/ridgeback_plus/urdf/ridgeback_plus.urdf.xacro (robot description, xacro)
@@ -8,4 +8,5 @@
        PosePublisher + legacy ign_ros2_control plugin) is skipped too. -->
   <xacro:arg name="use_platform_controllers" default="false"/>
+  <xacro:include filename="$(find clearpath_platform_description)/urdf/common.urdf.xacro"/>
   <xacro:include filename="$(find clearpath_platform_description)/urdf/r100/r100.urdf.xacro"/>
   <xacro:r100/>

File: arena_robots/arena_robots/robots/turtlebot/urdf/turtlebot.urdf.xacro (robot description, xacro)
@@ -1,4 +1,6 @@
 <?xml version="1.0"?>
 <robot name="turtlebot" xmlns:xacro="http://ros.org/wiki/xacro">
+  <xacro:arg name="namespace" default=""/>
+  <xacro:arg name="gazebo_controllers" default=""/>
   <!-- Base create3 model -->
   <xacro:include filename="$(find irobot_create_description)/urdf/create3.urdf.xacro">
@@ -11,4 +13,6 @@
   <xacro:include filename="$(find arena_robots)/robots/turtlebot/urdf/tower_sensor_plate.urdf.xacro" />
   <xacro:include filename="$(find arena_robots)/robots/turtlebot/urdf/weight_block.urdf.xacro" />
+  <xacro:include filename="$(find arena_robots)/robots/turtlebot/urdf/base_hw/turtlebot.ros2_control.urdf" />
+  <xacro:include filename="$(find arena_robots)/robots/turtlebot/urdf/turtlebot.gazebo" />
   <!-- Mechanical properties -->
   <xacro:property name="shell_z_offset"                value="${3*cm2m}" />
@@ -104,19 +108,5 @@
     <origin xyz="${oakd_pro_x_offset} ${oakd_pro_y_offset} ${oakd_pro_z_offset}"/>
   </xacro:oakd>
-  <!-- Gazebo Sim Plugins -->
-  <gazebo>
-    <plugin filename="gz-sim-joint-state-publisher-system" name="gz::sim::systems::JointStatePublisher">
-      <topic>joint_states</topic>
-    </plugin>
-    <plugin filename="gz-sim-diff-drive-system" name="gz::sim::systems::DiffDrive">
-      <left_joint>left_wheel_joint</left_joint>
-      <right_joint>right_wheel_joint</right_joint>
-      <wheel_separation>0.24</wheel_separation>
-      <wheel_radius>0.098</wheel_radius>
-      <odom_publish_frequency>50</odom_publish_frequency>
-      <!-- Suppress wheel-slip-polluted TF; pose_to_tf publishes odom→base_link from ground truth instead. -->
-      <tf_topic>/discard_tf</tf_topic>
-    </plugin>
-  </gazebo>
+  <xacro:turtlebot_base_hw_controller/>
   <!-- Wheel Friction and Dynamics -->
   <gazebo reference="wheel_left_link">
